Commit message: added lifespan to replace starutp handler, intermediate urdf folder backend upload

File: backend/temp_robot.urdf (robot description, URDF)
Before this commit: robot iiwa14, 9 links, 8 joints
Links:
- link link_0: geometry collision mesh filename=meshes/collision/link_0.obj; visual mesh filename=meshes/visual/link_0.obj
- link link_1: geometry collision mesh filename=meshes/collision/link_1.obj; visual mesh filename=meshes/visual/link_1.obj
- link link_2: geometry collision mesh filename=meshes/collision/link_2.obj; visual mesh filename=meshes/visual/link_2.obj
- link link_3: geometry collision mesh filename=meshes/collision/link_3.obj; visual mesh filename=meshes/visual/link_3.obj
- link link_4: geometry collision mesh filename=meshes/collision/link_4.obj; visual mesh filename=meshes/visual/link_4.obj
- link link_5: geometry collision mesh filename=meshes/collision/link_5.obj; visual mesh filename=meshes/visual/link_5.obj
- link link_6: geometry collision mesh filename=meshes/collision/link_6.obj; visual mesh filename=meshes/visual/link_6.obj
- link link_7: geometry collision mesh filename=meshes/collision/link_7.obj; visual mesh filename=meshes/visual/link_7.obj
